Commit message: Add crane_master_slave_control.launch

File: crane_plus_description/urdf/crane_plus.ros2_control.xacro (robot description, xacro)
@@ -1,4 +1,7 @@
 <?xml version="1.0"?>
 <robot xmlns:xacro="http://www.ros.org/wiki/xacro">
+  <xacro:property name="M_PI" value="3.14159"/>
+  <xacro:property name="TO_RADIAN" value="${M_PI / 180.0}"/>
+  <xacro:property name="X7_SERVO_HOME" value="${TO_RADIAN * 180.0}"/>
   <xacro:macro name="crane_plus_ros2_control_settings"
     params="name
@@ -86,4 +89,28 @@
       </joint>
     </ros2_control>
+    <ros2_control name="crane_x7" type="system">
+      <hardware>
+        <plugin>crane_x7_hardware/CraneX7Hardware</plugin>
+        <param name="port_name">/dev/ttyUSB1</param>
+        <param name="baudrate">3000000</param>
+        <param name="timeout_seconds">5.0</param>
+      </hardware>
+      <joint name="crane_x7_joint1">
+        <command_interface name="position">
+          <param name="min">"${90.0 * TO_RADIAN - X7_SERVO_HOME}"</param>
+          <param name="max">"${270.0 * TO_RADIAN - X7_SERVO_HOME}"</param>
+        </command_interface>
+        <state_interface name="position"/>
+        <param name="dxl_id">2</param>
+      </joint>
+      <!-- <joint name="crane_x7_joint2">
+        <command_interface name="position">
+          <param name="min">-1.57</param>
+          <param name="max">1.57</param>
+        </command_interface>
+        <state_interface name="position"/>
+        <param name="dxl_id">3</param>
+      </joint> -->
+    </ros2_control>
   </xacro:macro>
 </robot>

Commit message: Add inver_inputs option

File: crane_plus_description/urdf/crane_plus.ros2_control.xacro (robot description, xacro)
@@ -124,12 +124,28 @@
         <param name="dxl_id">2</param>
       </joint>
-      <!-- <joint name="crane_x7_joint2">
+      <joint name="crane_x7_joint2">
         <command_interface name="position">
-          <param name="min">-1.57</param>
-          <param name="max">1.57</param>
+          <param name="min">"${90.0 * TO_RADIAN - X7_SERVO_HOME}"</param>
+          <param name="max">"${270.0 * TO_RADIAN - X7_SERVO_HOME}"</param>
         </command_interface>
         <state_interface name="position"/>
         <param name="dxl_id">3</param>
-      </joint> -->
+      </joint>
+      <joint name="crane_x7_joint3">
+        <command_interface name="position">
+          <param name="min">"${90.0 * TO_RADIAN - X7_SERVO_HOME}"</param>
+          <param name="max">"${270.0 * TO_RADIAN - X7_SERVO_HOME}"</param>
+        </command_interface>
+        <state_interface name="position"/>
+        <param name="dxl_id">4</param>
+      </joint>
+      <joint name="crane_x7_joint4">
+        <command_interface name="position">
+          <param name="min">"${150.0 * TO_RADIAN - X7_SERVO_HOME}"</param>
+          <param name="max">"${0.0 * TO_RADIAN - X7_SERVO_HOME}"</param>
+        </command_interface>
+        <state_interface name="position"/>
+        <param name="dxl_id">5</param>
+      </joint>
     </ros2_control>
   </xacro:macro>

Commit message: add all joints of crane_x7

File: crane_plus_description/urdf/crane_plus.ros2_control.xacro (robot description, xacro)
@@ -148,4 +148,36 @@
         <param name="dxl_id">5</param>
       </joint>
+      <joint name="crane_x7_joint5">
+        <command_interface name="position">
+          <param name="min">"${90.0 * TO_RADIAN - X7_SERVO_HOME}"</param>
+          <param name="max">"${270.0 * TO_RADIAN - X7_SERVO_HOME}"</param>
+        </command_interface>
+        <state_interface name="position"/>
+        <param name="dxl_id">6</param>
+      </joint>
+      <joint name="crane_x7_joint6">
+        <command_interface name="position">
+          <param name="min">"${90.0 * TO_RADIAN - X7_SERVO_HOME}"</param>
+          <param name="max">"${270.0 * TO_RADIAN - X7_SERVO_HOME}"</param>
+        </command_interface>
+        <state_interface name="position"/>
+        <param name="dxl_id">7</param>
+      </joint>
+      <joint name="crane_x7_joint7">
+        <command_interface name="position">
+          <param name="min">"${90.0 * TO_RADIAN - X7_SERVO_HOME}"</param>
+          <param name="max">"${270.0 * TO_RADIAN - X7_SERVO_HOME}"</param>
+        </command_interface>
+        <state_interface name="position"/>
+        <param name="dxl_id">8</param>
+      </joint>
+      <joint name="crane_x7_joint_hand">
+        <command_interface name="position">
+          <param name="min">"${0.0 * TO_RADIAN - X7_SERVO_HOME}"</param>
+          <param name="max">"${90.0 * TO_RADIAN - X7_SERVO_HOME}"</param>
+        </command_interface>
+        <state_interface name="position"/>
+        <param name="dxl_id">9</param>
+      </joint>
     </ros2_control>
   </xacro:macro>
